Commit message: 20241181

File: manipulation_environment/urdf/environment_a.xacro (robot description, xacro)
@@ -4,25 +4,35 @@
   <link name="world" />
   <!-- world to world_interface. -->
+  <!--
   <joint name="world_to_world_interface" type="fixed">
     <parent link="world" />
     <child link="world_interface" />
   </joint>
+  -->
   <!-- workcell -->
+  <!--
   <xacro:include filename="$(find ros_industrial_support)/urdf/workshop/workshop.urdf.xacro"/>
   <xacro:workshop_urdf workshop_parent="world"/>
+  -->
   <!-- hall -->
+  <!--
   <xacro:include filename="$(find ros_industrial_support)/urdf/hall/hall.urdf.xacro"/>
   <xacro:hall_urdf hall_prefix="hall_" hall_parent="world">
     <origin xyz="-2.5 0 0.0" rpy="0 0 0"/>
   </xacro:hall_urdf>
+  -->
+  <xacro:include filename="$(find ros_industrial_support)/urdf/assembly_station/assembly_station.urdf.xacro"/>
+  <xacro:assembly_station_urdf assembly_station_prefix="shelf_" assembly_station_parent="world">
+    <origin xyz="1 0 0.0" rpy="0 0 ${radians(180)}"/>
+  </xacro:assembly_station_urdf>
   <!-- Mobile Computer -->
   <xacro:include filename="$(find ros_industrial_support)/urdf/computer_mobile/computer.urdf.xacro"/>
   <xacro:computer_urdf computer_parent="world" computer_prefix="comp_mobile_" >
-  <origin xyz="-5 0 0" rpy="0 0 2.1"/>
+  <origin xyz="-1.5 0 0" rpy="0 0 2.1"/>
   </xacro:computer_urdf>
   <!-- Robot1 Pedestal -->
   <xacro:include filename="$(find ros_industrial_support)/urdf/robot_pedestal/robot_pedestal.urdf.xacro"/>
-  <xacro:robot_pedestal_urdf pedestal_prefix="robot1_" pedestal_parent="world" pedestal_height="0.95">
-    <origin xyz="-4 -1 0.0" rpy="0 0 0"/>
+  <xacro:robot_pedestal_urdf pedestal_prefix="robot1_" pedestal_parent="world" pedestal_height="1.15">
+    <origin xyz="-0.5 -1 0.0" rpy="0 0 0"/>
   </xacro:robot_pedestal_urdf>
  <!-- Robot1 -->
@@ -36,7 +46,6 @@
   <xacro:bin_urdf prefix="bin_1_"/>
   <!-- robot1 to pedestal. -->
-  <!-- robot1 to pedestal. -->
   <joint name="robot1_to_pedestal" type="fixed">
-    <origin xyz="0 0 0.95" rpy="0 0 ${radians(90)}" />
+    <origin xyz="0 0 1.15" rpy="0 0 ${radians(90)}" />
     <parent link="robot1_pedestal_link" />
     <child link="robot1_xarm_link" />
@@ -51,5 +60,5 @@
     <parent link="world" />
     <child link="bin_1_base_link" />
-    <origin xyz="-4 -2 0.0" rpy="0 0 0" />
+    <origin xyz="-1.5 -2 0.0" rpy="0 0 0" />
   </joint>
 </robot>
