Commit message: 20241118-2

File: manipulation_environment/urdf/environment.xacro (robot description, xacro)
@@ -24,15 +24,15 @@
   <xacro:include filename="$(find ros_industrial_support)/urdf/assembly_station/assembly_station.urdf.xacro"/>
   <xacro:assembly_station_urdf assembly_station_prefix="shelf_" assembly_station_parent="world">
-    <origin xyz="1 0 0.0" rpy="0 0 ${radians(180)}"/>
+    <origin xyz="0.5 0.5 0.0" rpy="0 0 ${radians(180)}"/>
   </xacro:assembly_station_urdf>
   <!-- Mobile Computer -->
   <xacro:include filename="$(find ros_industrial_support)/urdf/computer_mobile/computer.urdf.xacro"/>
   <xacro:computer_urdf computer_parent="world" computer_prefix="comp_mobile_" >
-  <origin xyz="-1.5 0 0" rpy="0 0 2.1"/>
+  <origin xyz="0 1.5 0" rpy="0 0 2.1"/>
   </xacro:computer_urdf>
   <!-- Robot1 Pedestal -->
   <xacro:include filename="$(find ros_industrial_support)/urdf/robot_pedestal/robot_pedestal.urdf.xacro"/>
   <xacro:robot_pedestal_urdf pedestal_prefix="robot1_" pedestal_parent="world" pedestal_height="1.15">
-    <origin xyz="-0.5 -1 0.0" rpy="0 0 0"/>
+    <origin xyz="-0.0 0 0.0" rpy="0 0 0"/>
   </xacro:robot_pedestal_urdf>
  <!-- Robot1 -->
@@ -49,5 +49,5 @@
     <origin xyz="0 0 1.15" rpy="0 0 ${radians(90)}" />
     <parent link="robot1_pedestal_link" />
-    <child link="robot1_xarm_link" />
+    <child link="robot1_base_link" />
   </joint>
   <!-- gripper1 to robot1. -->
@@ -60,5 +60,5 @@
     <parent link="world" />
     <child link="bin_1_base_link" />
-    <origin xyz="-1.5 -2 0.0" rpy="0 0 0" />
+    <origin xyz="-0.5 -0.5 0.0" rpy="0 0 0" />
   </joint>
 </robot>
