Commit message: 20241122

File: manipulation_environment/urdf/environment.urdf.xacro (robot description, xacro)
@@ -26,5 +26,5 @@
  <!-- Robot1 -->
   <xacro:include filename="$(find ros_industrial_support)/urdf/ufactory/ufactory_xarm6.urdf.xacro"/>
-  <xacro:ufactory_xarm6 prefix="robot1_" joint_limited="true"/>
+  <xacro:ufactory_xarm6 prefix="" joint_limited="true"/>
   <!-- Vacuum Gripper1 -->
   <xacro:include filename="$(find ros_industrial_support)/urdf/vacuum_gripper/vacuum_gripper.urdf.xacro"/>
@@ -43,9 +43,9 @@
     <origin xyz="0 0 1.15" rpy="0 0 ${radians(0)}" />
     <parent link="robot1_pedestal_link" />
-    <child link="robot1_base_link" />
+    <child link="base_link" />
   </joint>
   <!-- gripper1 to robot1. -->
   <joint name="gripper1_to_robot1" type="fixed">
-    <parent link="robot1_tool_link" />
+    <parent link="tool_link" />
     <child link="vacuum_gripper1_base_link" />
   </joint>

File: manipulation_moveit_config/config/manipuation_environment.ros2_control.xacro (robot description, xacro)
@@ -8,43 +8,43 @@
                 <plugin>mock_components/GenericSystem</plugin>
             </hardware>
-            <joint name="robot1_joint1">
+            <joint name="joint1">
                 <command_interface name="position"/>
                 <state_interface name="position">
-                  <param name="initial_value">${initial_positions['robot1_joint1']}</param>
+                  <param name="initial_value">${initial_positions['joint1']}</param>
                 </state_interface>
                 <state_interface name="velocity"/>
             </joint>
-            <joint name="robot1_joint2">
+            <joint name="joint2">
                 <command_interface name="position"/>
                 <state_interface name="position">
-                  <param name="initial_value">${initial_positions['robot1_joint2']}</param>
+                  <param name="initial_value">${initial_positions['joint2']}</param>
                 </state_interface>
                 <state_interface name="velocity"/>
             </joint>
-            <joint name="robot1_joint3">
+            <joint name="joint3">
                 <command_interface name="position"/>
                 <state_interface name="position">
-                  <param name="initial_value">${initial_positions['robot1_joint3']}</param>
+                  <param name="initial_value">${initial_positions['joint3']}</param>
                 </state_interface>
                 <state_interface name="velocity"/>
             </joint>
-            <joint name="robot1_joint4">
+            <joint name="joint4">
                 <command_interface name="position"/>
                 <state_interface name="position">
-                  <param name="initial_value">${initial_positions['robot1_joint4']}</param>
+                  <param name="initial_value">${initial_positions['joint4']}</param>
                 </state_interface>
                 <state_interface name="velocity"/>
             </joint>
-            <joint name="robot1_joint5">
+            <joint name="joint5">
                 <command_interface name="position"/>
                 <state_interface name="position">
-                  <param name="initial_value">${initial_positions['robot1_joint5']}</param>
+                  <param name="initial_value">${initial_positions['joint5']}</param>
                 </state_interface>
                 <state_interface name="velocity"/>
             </joint>
-            <joint name="robot1_joint6">
+            <joint name="joint6">
                 <command_interface name="position"/>
                 <state_interface name="position">
-                  <param name="initial_value">${initial_positions['robot1_joint6']}</param>
+                  <param name="initial_value">${initial_positions['joint6']}</param>
                 </state_interface>
                 <state_interface name="velocity"/>

File: manipulation_moveit_config/config/manipuation_environment.urdf.xacro (robot description, xacro)
@@ -3,5 +3,5 @@
     <xacro:arg name="initial_positions_file" default="initial_positions.yaml" />
     <!-- Import manipuation_environment urdf file -->
-    <xacro:include filename="$(find manipulation_environment)/urdf/environment.xacro" />
+    <xacro:include filename="$(find manipulation_environment)/urdf/environment.urdf.xacro" />
     <!-- Import control_xacro -->
     <xacro:include filename="manipuation_environment.ros2_control.xacro" />
